File: spidebug.sch (KiCad schematic (older format))
At the start: 31 parts, among them P101 CONN_01X02, P102 CONN_01X02, P103 CONN_01X08, SW101 DPST 4A, SW102 SPDT 200mA, SW103 SW_PUSH, SW104 SW_PUSH, SW105 SW_PUSH, SW106 SW_PUSH

Commit message: Many small improvements.
* Move to V1.1 using less glue logic in the 7-seg display controller.

* Complete perfboard wiring diagram, show in layers.

* Minor spelling error and formatting improvements.
Changed lines of the file:
@@
 F 1 "DPST 4A" H 3700 3250 50  0000 C CNN
 F 2 "Wire_Pads:SolderWirePad_4xSquare_0-8mmDrill" H 3400 3300 50  0001 C CNN
-F 3 "https://www.ckswitches.com/media/1423/l.pdf" H 3400 3300 50  0000 C CNN
+F 3 "https://www.ckswitches.com/media/1423/l.pdf" H 3400 3300 50  0001 C CNN
 F 4 "CKN11876-ND" H 3400 3300 60  0001 C CNN "Digi-Key_PN"
 F 5 "L201011MS02Q" H 3400 3300 60  0001 C CNN "MPN"

Commit message: Improve switch footprints, add beveled 3D model.
Parts:
- SW101: footprint Wire_Pads:SolderWirePad_4xSquare_0-8mmDrill -> rpihw:Hack_L201
- SW102: footprint Wire_Pads:SolderWirePad_3x_0-8mmDrill -> Buttons_Switches_ThroughHole:SW_Micro_SPST
Changed lines of the file:
@@
 F 0 "SW101" H 3700 3350 50  0000 C CNN
 F 1 "DPST 4A" H 3700 3250 50  0000 C CNN
-F 2 "Wire_Pads:SolderWirePad_4xSquare_0-8mmDrill" H 3400 3300 50  0001 C CNN
+F 2 "rpihw:Hack_L201" H 3400 3300 50  0001 C CNN
 F 3 "https://www.ckswitches.com/media/1423/l.pdf" H 3400 3300 50  0001 C CNN
 F 4 "CKN11876-ND" H 3400 3300 60  0001 C CNN "Digi-Key_PN"
@@
 F 0 "SW102" H 5600 3450 50  0000 C CNN
 F 1 "SPDT 200mA" H 5650 3150 50  0000 C CNN
-F 2 "Wire_Pads:SolderWirePad_3x_0-8mmDrill" H 5800 3300 50  0001 C CNN
+F 2 "Buttons_Switches_ThroughHole:SW_Micro_SPST" H 5800 3300 50  0001 C CNN
 F 3 "https://sten-eswitch-13110800-production.s3.amazonaws.com/system/asset/product_line/data_sheet/119/EG.pdf" H 5800 3300 50  0001 C CNN
 F 4 "EG1903-ND" H 5800 3300 60  0001 C CNN "Digi-Key_PN"
