File: rpihw.kicad_pcb (KiCad board)
At the start: 4 copper layers, 207 x 78.7 mm, 101 parts, among them P1 CONN_01X02, P101 CONN_01X02, P102 CONN_01X02, P103 CONN_01X08, P2 CONN_01X02, P3 CONN_02X20, Q1 2N3904BU, Q2 2N3904BU, Q3 2N3904BU, Q4 2N3904BU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

Commit message: Improve footprint hole diameters, add DO-201AD 3D model.
Also use two-sided layers setup since through-hole boards need solder
mask on both sides.
Parts:
- moved SW1 0.63 mm to (146.1, 97.8)

Commit message: Better silkscreen, footprint corrections.
Parts:
- moved C13 2.54 mm to (90.2, 104.1)
- moved P1 2.54 mm to (135.9, 95.2), turned to 180 degrees
- moved P2 2.54 mm to (135.9, 102.9), turned to 180 degrees
Routing:
- net /SPI 7-SEG DPLY KEYPAD CTL DIP/VCC: track 309.3 -> 581.2 mm, vias 2 -> 5
- net /SPI MOTOR CTL DIP/VS: track 156.8 -> 207.3 mm, vias 2 -> 4
- net /RPI SPI BOARD DIP/GND_MTR: track 67.3 -> 84.8 mm
- net Net-(P1-Pad1): track 31.1 -> 13.8 mm
- net Net-(D1-Pad2): track 46.7 -> 52.3 mm
- net Net-(P2-Pad1): track 16.6 -> 13.8 mm, vias 1 -> 0
- net Net-(D2-Pad2): track 86.1 -> 87.2 mm

Commit message: Improve footprints, add 3D model for big TVS diode.
Whoops, I didn't checkin the earlier revision switch footprints, those
revisions will be broken unfortunately.
Parts:
- D2: footprint Diodes_ThroughHole:Diode_DO-201AD_Horizontal_RM15 -> rpihw:Diode_R-6_Horizontal_Unpol_RM15
- moved SW101 5.68 mm to (191.8, 94.0)
- moved SW1 2.54 mm to (146.1, 100.3)
